Commit message: Salva modifiche locali su Real

File: src/scooby_description/urdf/lidar_gazebo_macro.xacro (robot description, xacro)
@@ -2,5 +2,5 @@
 <robot xmlns:xacro="http://www.ros.org/wiki/xacro" name="lidar_gazebo_macro" >
   <!--xacro:include filename="$(find scooby_description)/urdf/utility_macro.xacro" /-->
-  <xacro:macro name="lidar_gazebo_sensor" params="parent">
+  <xacro:macro name="lidar_gazebo_sensor" params="name:=lidar parent *origin">
     <!-- Lidar is composed by a single link and a fixed joint -->
     <link name="laser_frame">
@@ -27,5 +27,5 @@
       <parent link="${parent}" />
       <child link="laser_frame" />
-      <origin rpy="0 0 0" xyz="0.0 0.0 0.031" />
+      <xacro:insert_block name="origin" />
     </joint>
     <!-- Gazebo plugin for the LiDAR sensor -->

File: src/scooby_description/urdf/scooby.urdf.xacro (robot description, xacro)
@@ -4,18 +4,20 @@
 <robot xmlns:xacro="http://www.ros.org/wiki/xacro" name="scooby" >
   <xacro:include filename="$(find scooby_description)/urdf/scooby_base_macro.xacro"/>
-  <!--xacro:include filename="$(find scooby_description)/urdf/lidar_gazebo_macro.xacro"/>
-  <xacro:include filename="$(find scooby_description)/urdf/d435_gazebo_macro.xacro" />
+  <xacro:include filename="$(find scooby_description)/urdf/lidar_gazebo_macro.xacro"/>
+  <xacro:include filename="$(find scooby_description)/urdf/camera.xacro" />
+  <xacro:property name="CAMERA" value="True"/>
   <xacro:property name="LIDAR" value="True"/>
-  <xacro:property name="DEPTH" value="True"/>
-  -->
   <!-- Diff Drive Robot Base -->
   <xacro:scooby_base/>
-  <!-- LIDAR Sensor-->
-  <!--xacro:if value="${LIDAR}">
-    <xacro:lidar_gazebo_sensor parent="lidar_link"/>
-  </xacro:if-->
-  <!-- RGBD Sensor (D435 Camera) -->
-  <!--xacro:if value="${DEPTH}">
-    <xacro:d435_gazebo_sensor parent="d435_link" />
-  </xacro:if-->
+  <!-- LIDAR Sensor -->
+  <xacro:if value="${LIDAR}">
+    <xacro:lidar_gazebo_sensor name="lidar_gazebo_macro" parent="lidar_link">
+      <origin xyz="0.0 0.0 0.031" rpy="0 0 0" />
+    </xacro:lidar_gazebo_sensor>
+  </xacro:if>
+  <xacro:if value="${CAMERA}">
+    <xacro:scooby_rgbd_camera name="camera" parent="d435_link">
+      <origin xyz="0 0 0" rpy="0 0 0" />
+    </xacro:scooby_rgbd_camera>
+  </xacro:if>
 </robot>

File: src/scooby_description/urdf/scooby_base_macro.xacro (robot description, xacro)
@@ -172,5 +172,5 @@
       <parent link="base_footprint" />
       <child link="base_link" />
-      <origin xyz="0.0 0.0 ${0.059 + body_z_offset}" rpy="0 0 0" />
+      <origin xyz="0.0 0.0 ${0.059 + body_z_offset}" rpy="0 0 ${-M_PI_2}" />
     </joint>
     <!-- Joint: sinistra (motrice) -->
@@ -195,10 +195,10 @@
       <parent link="base_link" />
       <child link="d435_link" />
-      <origin xyz="0.090925 0.0 0.06670" rpy="0 0 0" />
+      <origin xyz="0.07 0.0 0.0" rpy="0 0 0" />
     </joint>
     <joint name="lidar_joint" type="fixed">
       <parent link="base_link" />
       <child link="lidar_link" />
-      <origin xyz="0.0 0.0 0.125" rpy="0 0 0" />
+      <origin xyz="0.0 0.0 0.05" rpy="0 0 0" />
     </joint>
     <!-- Transmissions solo per le ruote motrici -->
