Commit message: Aggiornamento file e push modifiche

File: src/scooby_description/urdf/scooby_base_macro.xacro (robot description, xacro)
@@ -5,73 +5,121 @@
   <!-- Odometry root frame -->
   <link name="base_footprint"/>
-    <!-- Base properties -->
-    <xacro:property name="base_height" value="0.180" />
-    <xacro:property name="base_radius" value="0.11" />
+    <!-- Base properties (box: 0.13 x 0.09 x 0.11 m) -->
+    <xacro:property name="base_length" value="0.13" /> <!-- X -->
+    <xacro:property name="base_width" value="0.09" />  <!-- Y -->
+    <xacro:property name="base_height" value="0.11" /> <!-- Z -->
     <xacro:property name="base_mass" value="5" />
+    <!-- Wheel properties (cylinder: r=0.03, l=0.04) -->
+    <xacro:property name="wheel_radius" value="0.03" />
+    <xacro:property name="wheel_length" value="0.04" />
     <xacro:property name="wheel_mass" value="2.5" />
-    <xacro:property name="wheel_radius" value="0.035" />
-    <xacro:property name="wheel_axle" value="0.13" />
+    <!-- Wheel separation (distanza tra i centri delle ruote su y) -->
+    <xacro:property name="wheel_separation" value="0.14" />
+    <!-- Wheel longitudinal offset (distanza tra asse centrale e ruote anteriori/posteriori su x) -->
+    <xacro:property name="wheel_x_offset" value="0.075" />
     <link name="base_link">
-      <!-- Inertial properties -->
+      <!-- Inertial properties: parallelepipedo 0.13x0.09x0.11 -->
       <inertial>
         <origin xyz="0 0 0" />
         <mass value="${base_mass}" />
-        <xacro:cylinder_inertia m="${base_mass}" r="${base_radius}" h="${base_height}" />
-      </inertial>
-      <!-- Visual representation -->
-      <visual>
-        <geometry>
-          <mesh filename="file://$(find scooby_description)/meshes/scooby_body.stl" scale="0.001 0.001 0.001" />
+        <inertia
+          ixx="${(1/12.0)*base_mass*(base_width*base_width + base_height*base_height)}"
+          ixy="0.0" ixz="0.0"
+          iyy="${(1/12.0)*base_mass*(base_length*base_length + base_height*base_height)}"
+          iyz="0.0"
+          izz="${(1/12.0)*base_mass*(base_length*base_length + base_width*base_width)}" />
+        <!-- Calcolato per box: ixx = 1/12*m*(y^2+z^2), iyy = 1/12*m*(x^2+z^2), izz = 1/12*m*(x^2+y^2) -->
+      </inertial>
+      <!-- Visual representation: parallelepipedo 13x9x11 cm (inverto x e y) -->
+      <visual>
+        <geometry>
+          <box size="${base_length} ${base_width} ${base_height}" />
         </geometry>
         <material name="Blue" />
         <origin xyz="0 0 0" rpy="0 0 0" />
       </visual>
-      <!-- Collision properties -->
-      <collision>
-        <geometry>
-          <cylinder length="${base_height}" radius="${base_radius}" />
-        </geometry>
-        <origin xyz="0 0.0 ${(base_height/2.0)-0.05}" rpy="0 0 0" />
-      </collision>
-      <collision>
-        <geometry>
-          <sphere radius="0.019" />
-        </geometry>
-        <origin xyz="-0.0825 0.0 -0.04" rpy="0 0 0" />
-      </collision>
-    </link>
-    <!-- Left Wheel -->
-    <link name="left_wheel_link">
-      <visual>
-        <geometry>
-          <mesh filename="file://$(find scooby_description)/meshes/scooby_wheel.stl" scale="0.001 0.001 0.001" />
-        </geometry>
-        <material name="Black" />
+      <!-- Collision properties: parallelepipedo 0.13x0.09x0.11 -->
+      <collision>
+        <geometry>
+          <box size="${base_length} ${base_width} ${base_height}" />
+        </geometry>
         <origin xyz="0 0 0" rpy="0 0 0" />
-      </visual>
-      <collision>
-        <geometry>
-          <cylinder length="0.02" radius="${wheel_radius}" />
-        </geometry>
-        <origin xyz="0 0 0" rpy="0 1.5708 1.5708" />
-      </collision>
-      <inertial>
-        <origin xyz="0 0 0" />
-        <mass value="${wheel_mass}" />
-        <inertia ixx="0.001" ixy="0.0" ixz="0.0" iyy="0.001" iyz="0.0" izz="0.001" />
-      </inertial>
-    </link>
-    <!-- Right Wheel -->
-    <link name="right_wheel_link">
-      <visual>
-        <geometry>
-          <mesh filename="file://$(find scooby_description)/meshes/scooby_wheel.stl" scale="0.001 0.001 0.001" />
-        </geometry>
-        <material name="Black"/>
-        <origin xyz="0 0 0" rpy="0 0 0" />
-      </visual>
-      <collision>
-        <geometry>
-          <cylinder length="0.02" radius="${wheel_radius}" />
+      </collision>
+    </link>
+    <!-- Motrice: Anteriore Sinistra -->
+    <link name="left_wheel_link_f">
+      <visual>
+        <geometry>
+          <cylinder length="${wheel_length}" radius="${wheel_radius}" />
+        </geometry>
+        <material name="Black" />
+        <origin xyz="0 0 0" rpy="0 1.5708 1.5708" />
+      </visual>
+      <collision>
+        <geometry>
+          <cylinder length="${wheel_length}" radius="${wheel_radius}" />
+        </geometry>
+        <origin xyz="0 0 0" rpy="0 1.5708 1.5708" />
+      </collision>
+      <inertial>
+        <origin xyz="0 0 0" />
+        <mass value="${wheel_mass}" />
+        <inertia ixx="0.001" ixy="0.0" ixz="0.0" iyy="0.001" iyz="0.0" izz="0.001" />
+      </inertial>
+    </link>
+    <!-- Passiva: Posteriore Sinistra -->
+    <link name="left_wheel_link_b">
+      <visual>
+        <geometry>
+          <cylinder length="${wheel_length}" radius="${wheel_radius}" />
+        </geometry>
+        <material name="Black" />
+        <origin xyz="0 0 0" rpy="0 1.5708 1.5708" />
+      </visual>
+      <collision>
+        <geometry>
+          <cylinder length="${wheel_length}" radius="${wheel_radius}" />
+        </geometry>
+        <origin xyz="0 0 0" rpy="0 1.5708 1.5708" />
+      </collision>
+      <inertial>
+        <origin xyz="0 0 0" />
+        <mass value="${wheel_mass}" />
+        <inertia ixx="0.001" ixy="0.0" ixz="0.0" iyy="0.001" iyz="0.0" izz="0.001" />
+      </inertial>
+    </link>
+    <!-- Passiva: Anteriore Destra -->
+    <link name="right_wheel_link_f">
+      <visual>
+        <geometry>
+          <cylinder length="${wheel_length}" radius="${wheel_radius}" />
+        </geometry>
+        <material name="Black" />
+        <origin xyz="0 0 0" rpy="0 1.5708 1.5708" />
+      </visual>
+      <collision>
+        <geometry>
+          <cylinder length="${wheel_length}" radius="${wheel_radius}" />
+        </geometry>
+        <origin xyz="0 0 0" rpy="0 1.5708 1.5708" />
+      </collision>
+      <inertial>
+        <origin xyz="0 0 0" />
+        <mass value="${wheel_mass}" />
+        <inertia ixx="0.001" ixy="0.0" ixz="0.0" iyy="0.001" iyz="0.0" izz="0.001" />
+      </inertial>
+    </link>
+    <!-- Motrice: Posteriore Destra -->
+    <link name="right_wheel_link_b">
+      <visual>
+        <geometry>
+          <cylinder length="${wheel_length}" radius="${wheel_radius}" />
+        </geometry>
+        <material name="Black" />
+        <origin xyz="0 0 0" rpy="0 1.5708 1.5708" />
+      </visual>
+      <collision>
+        <geometry>
+          <cylinder length="${wheel_length}" radius="${wheel_radius}" />
         </geometry>
         <origin xyz="0 0 0" rpy="0 1.5708 1.5708" />
@@ -93,16 +141,36 @@
       <origin xyz="0.0 0.0 0.059" rpy="0 0 0" />
     </joint>
-    <joint name="left_wheel_joint" type="continuous">
-      <parent link="base_link" />
-      <child link="left_wheel_link" />
-      <origin xyz="0.04025 0.062 -0.024" rpy="0 0 0" />
+    <!-- Motrice: Anteriore Sinistra -->
+    <joint name="left_wheel_joint_f" type="continuous">
+      <parent link="base_link" />
+      <child link="left_wheel_link_f" />
+      <origin xyz="${wheel_x_offset} ${wheel_separation/2.0} -0.024" rpy="0 0 0" />
       <axis xyz="0 1 0" />
       <limit effort="100" velocity="100" />
       <dynamics damping="0.5" friction="0.01" />
     </joint>
-    <joint name="right_wheel_joint" type="continuous">
-      <parent link="base_link" />
-      <child link="right_wheel_link" />
-      <origin xyz="0.04025 -0.062 -0.024" rpy="0 0 ${-M_PI}" />
+    <!-- Motrice: Posteriore Destra -->
+    <joint name="right_wheel_joint_b" type="continuous">
+      <parent link="base_link" />
+      <child link="right_wheel_link_b" />
+      <origin xyz="-${wheel_x_offset} -${wheel_separation/2.0} -0.024" rpy="0 0 ${-M_PI}" />
+      <axis xyz="0 -1 0" />
+      <limit effort="100" velocity="100" />
+      <dynamics damping="0.5" friction="0.01" />
+    </joint>
+    <!-- Passiva: Posteriore Sinistra -->
+    <joint name="left_wheel_joint_b" type="continuous">
+      <parent link="base_link" />
+      <child link="left_wheel_link_b" />
+      <origin xyz="-${wheel_x_offset} ${wheel_separation/2.0} -0.024" rpy="0 0 0" />
+      <axis xyz="0 1 0" />
+      <limit effort="100" velocity="100" />
+      <dynamics damping="0.5" friction="0.01" />
+    </joint>
+    <!-- Passiva: Anteriore Destra -->
+    <joint name="right_wheel_joint_f" type="continuous">
+      <parent link="base_link" />
+      <child link="right_wheel_link_f" />
+      <origin xyz="${wheel_x_offset} -${wheel_separation/2.0} -0.024" rpy="0 0 ${-M_PI}" />
       <axis xyz="0 -1 0" />
       <limit effort="100" velocity="100" />
@@ -120,16 +188,16 @@
     </joint>
     <!-- Transmissions for the wheel joints -->
-    <transmission name="left_wheel_joint_trans">
+    <transmission name="left_wheel_joint_f_trans">
       <type>transmission_interface/SimpleTransmission</type>
-      <joint name="left_wheel_joint" />
-      <actuator name="left_wheel_joint_motor">
+      <joint name="left_wheel_joint_f" />
+      <actuator name="left_wheel_joint_f_motor">
         <mechanicalReduction>1</mechanicalReduction>
         <hardwareInterface>EffortJointInterface</hardwareInterface>
       </actuator>
     </transmission>
-    <transmission name="right_wheel_joint_trans">
+    <transmission name="right_wheel_joint_b_trans">
       <type>transmission_interface/SimpleTransmission</type>
-      <joint name="right_wheel_joint" />
-      <actuator name="right_wheel_joint_motor">
+      <joint name="right_wheel_joint_b" />
+      <actuator name="right_wheel_joint_b_motor">
         <mechanicalReduction>1</mechanicalReduction>
         <hardwareInterface>EffortJointInterface</hardwareInterface>
@@ -138,10 +206,11 @@
     <!-- Plugin for differential drive control in Gazebo-->
     <gazebo>
+      <!-- Plugin per 4 ruote: puoi sostituire con un plugin custom se necessario -->
       <plugin
         filename="libgz-sim-diff-drive-system.so"
         name="gz::sim::systems::DiffDrive">
-        <left_joint>left_wheel_joint</left_joint>
-        <right_joint>right_wheel_joint</right_joint>
-        <wheel_separation>${wheel_axle}</wheel_separation>
+        <left_joint>left_wheel_joint_f</left_joint>
+        <right_joint>right_wheel_joint_b</right_joint>
+        <wheel_separation>${wheel_separation}</wheel_separation>
         <wheel_radius>${wheel_radius}</wheel_radius>
         <!-- Limits for the differential drive -->
@@ -170,6 +239,8 @@
         name="gz::sim::systems::JointStatePublisher">
         <topic>/joint_states</topic>
-        <joint_name>left_wheel_joint</joint_name>
-        <joint_name>right_wheel_joint</joint_name>
+        <joint_name>left_wheel_joint_f</joint_name>
+        <joint_name>right_wheel_joint_b</joint_name>
+        <joint_name>left_wheel_joint_b</joint_name>
+        <joint_name>right_wheel_joint_f</joint_name>
       </plugin>
     </gazebo>

Commit message: Aggiornamento file e push modifiche

File: src/scooby_description/urdf/scooby_base_macro.xacro (robot description, xacro)
@@ -7,6 +7,6 @@
     <!-- Base properties (box: 0.13 x 0.09 x 0.11 m) -->
     <xacro:property name="base_length" value="0.13" /> <!-- X -->
-    <xacro:property name="base_width" value="0.09" />  <!-- Y -->
-    <xacro:property name="base_height" value="0.11" /> <!-- Z -->
+    <xacro:property name="base_width" value="0.11" />  <!-- Y -->
+    <xacro:property name="base_height" value="0.09" /> <!-- Z -->
     <xacro:property name="base_mass" value="5" />
     <!-- Wheel properties (cylinder: r=0.03, l=0.04) -->
@@ -18,6 +18,7 @@
     <!-- Wheel longitudinal offset (distanza tra asse centrale e ruote anteriori/posteriori su x) -->
     <xacro:property name="wheel_x_offset" value="0.075" />
+    <xacro:property name="body_z_offset" value="${base_height/2.0 + caster_radius}" /> <!-- base completamente sopra la sfera -->
+    <xacro:property name="caster_radius" value="0.018" /> <!-- raggio sfera caster -->
     <link name="base_link">
-      <!-- Inertial properties: parallelepipedo 0.13x0.09x0.11 -->
       <inertial>
         <origin xyz="0 0 0" />
@@ -29,7 +30,5 @@
           iyz="0.0"
           izz="${(1/12.0)*base_mass*(base_length*base_length + base_width*base_width)}" />
-        <!-- Calcolato per box: ixx = 1/12*m*(y^2+z^2), iyy = 1/12*m*(x^2+z^2), izz = 1/12*m*(x^2+y^2) -->
-      </inertial>
-      <!-- Visual representation: parallelepipedo 13x9x11 cm (inverto x e y) -->
+      </inertial>
       <visual>
         <geometry>
@@ -39,5 +38,4 @@
         <origin xyz="0 0 0" rpy="0 0 0" />
       </visual>
-      <!-- Collision properties: parallelepipedo 0.13x0.09x0.11 -->
       <collision>
         <geometry>
@@ -45,8 +43,86 @@
         </geometry>
         <origin xyz="0 0 0" rpy="0 0 0" />
-      </collision>
-    </link>
-    <!-- Motrice: Anteriore Sinistra -->
-    <link name="left_wheel_link_f">
+        <surface>
+          <friction>
+            <ode>
+              <mu>0.0</mu>
+              <mu2>0.0</mu2>
+            </ode>
+          </friction>
+        </surface>
+      </collision>
+    </link>
+              <!-- Caster wheel (sfera) sotto la base -->
+    <link name="caster_wheel_link1">
+      <visual>
+        <geometry>
+          <sphere radius="${caster_radius}" />
+        </geometry>
+        <material name="Grey" />
+        <origin xyz="0.02 0 -0.031" rpy="0 0 0" />
+      </visual>
+      <collision>
+        <geometry>
+          <sphere radius="${caster_radius}" />
+        </geometry>
+        <origin xyz="0.02 0 -0.031" rpy="0 0 0" />
+        <surface>
+          <friction>
+            <ode>
+              <mu>0.0</mu>
+              <mu2>0.0</mu2>
+            </ode>
+          </friction>
+        </surface>
+      </collision>
+      <inertial>
+        <origin xyz="0 0 0" />
+        <mass value="0.01" />
+        <inertia ixx="0.00001" ixy="0.0" ixz="0.0" iyy="0.00001" iyz="0.0" izz="0.00001" />
+      </inertial>
+    </link>
+    <!-- Joint fisso tra base e caster -->
+    <joint name="caster_wheel_joint1" type="fixed">
+      <parent link="base_link" />
+      <child link="caster_wheel_link1" />
+      <origin xyz="0.02 0 -0.031" rpy="0 0 0" />
+    </joint>
+                  <!-- Caster wheel (sfera) sotto la base -->
+    <link name="caster_wheel_link2">
+      <visual>
+        <geometry>
+          <sphere radius="${caster_radius}" />
+        </geometry>
+        <material name="Grey" />
+        <origin xyz="-0.02 0 -0.031" rpy="0 0 0" />
+      </visual>
+      <collision>
+        <geometry>
+          <sphere radius="${caster_radius}" />
+        </geometry>
+        <origin xyz="-0.02 0 -0.031" rpy="0 0 0" />
+        <surface>
+          <friction>
+            <ode>
+              <mu>0.0</mu>
+              <mu2>0.0</mu2>
+            </ode>
+          </friction>
+        </surface>
+      </collision>
+      <inertial>
+        <origin xyz="0 0 0" />
+        <mass value="0.01" />
+        <inertia ixx="0.00001" ixy="0.0" ixz="0.0" iyy="0.00001" iyz="0.0" izz="0.00001" />
+      </inertial>
+    </link>
+    <!-- Joint fisso tra base e caster -->
+    <joint name="caster_wheel_joint2" type="fixed">
+      <parent link="base_link" />
+      <child link="caster_wheel_link2" />
+      <origin xyz="-0.02 0 -0.031" rpy="0 0 0" />
+    </joint>
+    <!-- Ruote: anteriore motrici, posteriore passive -->
+    <link name="left_wheel_link">
       <visual>
         <geometry>
@@ -68,48 +144,5 @@
       </inertial>
     </link>
-    <!-- Passiva: Posteriore Sinistra -->
-    <link name="left_wheel_link_b">
-      <visual>
-        <geometry>
-          <cylinder length="${wheel_length}" radius="${wheel_radius}" />
-        </geometry>
-        <material name="Black" />
-        <origin xyz="0 0 0" rpy="0 1.5708 1.5708" />
-      </visual>
-      <collision>
-        <geometry>
-          <cylinder length="${wheel_length}" radius="${wheel_radius}" />
-        </geometry>
-        <origin xyz="0 0 0" rpy="0 1.5708 1.5708" />
-      </collision>
-      <inertial>
-        <origin xyz="0 0 0" />
-        <mass value="${wheel_mass}" />
-        <inertia ixx="0.001" ixy="0.0" ixz="0.0" iyy="0.001" iyz="0.0" izz="0.001" />
-      </inertial>
-    </link>
-    <!-- Passiva: Anteriore Destra -->
-    <link name="right_wheel_link_f">
-      <visual>
-        <geometry>
-          <cylinder length="${wheel_length}" radius="${wheel_radius}" />
-        </geometry>
-        <material name="Black" />
-        <origin xyz="0 0 0" rpy="0 1.5708 1.5708" />
-      </visual>
-      <collision>
-        <geometry>
-          <cylinder length="${wheel_length}" radius="${wheel_radius}" />
-        </geometry>
-        <origin xyz="0 0 0" rpy="0 1.5708 1.5708" />
-      </collision>
-      <inertial>
-        <origin xyz="0 0 0" />
-        <mass value="${wheel_mass}" />
-        <inertia ixx="0.001" ixy="0.0" ixz="0.0" iyy="0.001" iyz="0.0" izz="0.001" />
-      </inertial>
-    </link>
-    <!-- Motrice: Posteriore Destra -->
-    <link name="right_wheel_link_b">
+    <link name="right_wheel_link">
       <visual>
         <geometry>
@@ -139,42 +172,24 @@
       <parent link="base_footprint" />
       <child link="base_link" />
-      <origin xyz="0.0 0.0 0.059" rpy="0 0 0" />
-    </joint>
-    <!-- Motrice: Anteriore Sinistra -->
-    <joint name="left_wheel_joint_f" type="continuous">
-      <parent link="base_link" />
-      <child link="left_wheel_link_f" />
-      <origin xyz="${wheel_x_offset} ${wheel_separation/2.0} -0.024" rpy="0 0 0" />
+      <origin xyz="0.0 0.0 ${0.059 + body_z_offset}" rpy="0 0 0" />
+    </joint>
+    <!-- Joint: sinistra (motrice) -->
+    <joint name="left_wheel_joint" type="continuous">
+      <parent link="base_link" />
+      <child link="left_wheel_link" />
+      <origin xyz="0 ${wheel_separation/2.0} -0.05" rpy="0 0 0" />
       <axis xyz="0 1 0" />
       <limit effort="100" velocity="100" />
       <dynamics damping="0.5" friction="0.01" />
     </joint>
-    <!-- Motrice: Posteriore Destra -->
-    <joint name="right_wheel_joint_b" type="continuous">
-      <parent link="base_link" />
-      <child link="right_wheel_link_b" />
-      <origin xyz="-${wheel_x_offset} -${wheel_separation/2.0} -0.024" rpy="0 0 ${-M_PI}" />
+    <!-- Joint: destra (motrice) -->
+    <joint name="right_wheel_joint" type="continuous">
+      <parent link="base_link" />
+      <child link="right_wheel_link" />
+      <origin xyz="0 -${wheel_separation/2.0} -0.05" rpy="0 0 ${-M_PI}" />
       <axis xyz="0 -1 0" />
       <limit effort="100" velocity="100" />
       <dynamics damping="0.5" friction="0.01" />
     </joint>
-    <!-- Passiva: Posteriore Sinistra -->
-    <joint name="left_wheel_joint_b" type="continuous">
-      <parent link="base_link" />
-      <child link="left_wheel_link_b" />
-      <origin xyz="-${wheel_x_offset} ${wheel_separation/2.0} -0.024" rpy="0 0 0" />
-      <axis xyz="0 1 0" />
-      <limit effort="100" velocity="100" />
-      <dynamics damping="0.5" friction="0.01" />
-    </joint>
-    <!-- Passiva: Anteriore Destra -->
-    <joint name="right_wheel_joint_f" type="continuous">
-      <parent link="base_link" />
-      <child link="right_wheel_link_f" />
-      <origin xyz="${wheel_x_offset} -${wheel_separation/2.0} -0.024" rpy="0 0 ${-M_PI}" />
-      <axis xyz="0 -1 0" />
-      <limit effort="100" velocity="100" />
-      <dynamics damping="0.5" friction="0.01" />
-    </joint>
     <joint name="d435_joint" type="fixed">
       <parent link="base_link" />
@@ -187,17 +202,17 @@
       <origin xyz="0.0 0.0 0.125" rpy="0 0 0" />
     </joint>
-    <!-- Transmissions for the wheel joints -->
-    <transmission name="left_wheel_joint_f_trans">
+    <!-- Transmissions solo per le ruote motrici -->
+    <transmission name="left_wheel_joint_trans">
       <type>transmission_interface/SimpleTransmission</type>
-      <joint name="left_wheel_joint_f" />
-      <actuator name="left_wheel_joint_f_motor">
+      <joint name="left_wheel_joint" />
+      <actuator name="left_wheel_joint_motor">
         <mechanicalReduction>1</mechanicalReduction>
         <hardwareInterface>EffortJointInterface</hardwareInterface>
       </actuator>
     </transmission>
-    <transmission name="right_wheel_joint_b_trans">
+    <transmission name="right_wheel_joint_trans">
       <type>transmission_interface/SimpleTransmission</type>
-      <joint name="right_wheel_joint_b" />
-      <actuator name="right_wheel_joint_b_motor">
+      <joint name="right_wheel_joint" />
+      <actuator name="right_wheel_joint_motor">
         <mechanicalReduction>1</mechanicalReduction>
         <hardwareInterface>EffortJointInterface</hardwareInterface>
@@ -210,6 +225,6 @@
         filename="libgz-sim-diff-drive-system.so"
         name="gz::sim::systems::DiffDrive">
-        <left_joint>left_wheel_joint_f</left_joint>
-        <right_joint>right_wheel_joint_b</right_joint>
+        <left_joint>left_wheel_joint</left_joint>
+        <right_joint>right_wheel_joint</right_joint>
         <wheel_separation>${wheel_separation}</wheel_separation>
         <wheel_radius>${wheel_radius}</wheel_radius>
@@ -239,8 +254,6 @@
         name="gz::sim::systems::JointStatePublisher">
         <topic>/joint_states</topic>
-        <joint_name>left_wheel_joint_f</joint_name>
-        <joint_name>right_wheel_joint_b</joint_name>
-        <joint_name>left_wheel_joint_b</joint_name>
-        <joint_name>right_wheel_joint_f</joint_name>
+        <joint_name>left_wheel_joint</joint_name>
+        <joint_name>right_wheel_joint</joint_name>
       </plugin>
     </gazebo>

Commit message: Update navigation configs and launch files

File: src/scooby_description/urdf/scooby_base_macro.xacro (robot description, xacro)
@@ -172,5 +172,5 @@
       <parent link="base_footprint" />
       <child link="base_link" />
-      <origin xyz="0.0 0.0 ${0.059 + body_z_offset}" rpy="0 0 ${-M_PI_2}" />
+      <origin xyz="0.0 0.0 ${0.059 + body_z_offset}" rpy="0 0 ${M_PI_2}" />
     </joint>
     <!-- Joint: sinistra (motrice) -->
@@ -245,6 +245,6 @@
         <frame_id>odom</frame_id>
         <child_frame_id>base_footprint</child_frame_id>
-        <publish_odom>true</publish_odom>
-        <publish_odom_tf>true</publish_odom_tf>
+        <publish_odom>false</publish_odom>
+        <publish_odom_tf>false</publish_odom_tf>
         <publish_wheel_tf>true</publish_wheel_tf>
       </plugin>
